File: kicad/ESP-In-De_ThroughHole/ESP-In-De_ThroughHole.sch (KiCad schematic (older format))
At the start: 30 parts

Commit message: Schematic and Readme updates
- Created through-hole schematic with most basic functionality implemented - still need to add sync and onboard buttons
Parts:
- added J?: Player 1 Buttons, symbol ESP-In-De_Symbols:Conn_20_Pin_Joystick
- added J?: Player 2 Buttons, symbol ESP-In-De_Symbols:Conn_20_Pin_Joystick
- J?: value Player 1 Buttons -> Player 1 Buttons In
- J?: value Player 2 Buttons -> Player 2 Buttons In
Connections:
- net GND: now also J?.12 (GND), J?.12 (GND), J?.17 (GND), J?.17 (GND), J?.18 (GND), J?.18 (GND)
- net Out_P1_B1: now also J?.8 (1P)
- net Out_P1_B2: now also J?.9 (2P)
- net Out_P1_B3: now also J?.10 (3P)
- net Out_P1_B4: now also J?.13 (1K)
- net Out_P1_B5: now also J?.14 (2K)
- net Out_P1_B6: now also J?.15 (3K)
- net Out_P1_B7: now also J?.11 (4P)
- net Out_P1_B8: now also J?.16 (4K)
- net Out_P1_Down: now also J?.2 (Down)
- net Out_P1_Left: now also J?.4 (Left)
- net Out_P1_Right: now also J?.3 (Right)
- net Out_P1_Start: now also J?.7 (Start/Opt)
- net Out_P1_Up: now also J?.1 (Up)
- net Out_P2_B1: now also J?.8 (1P)
- net Out_P2_B2: now also J?.9 (2P)
- net Out_P2_B3: now also J?.10 (3P)
- net Out_P2_B4: now also J?.13 (1K)
- net Out_P2_B5: now also J?.14 (2K)
- net Out_P2_B6: now also J?.15 (3K)
- net Out_P2_B7: now also J?.11 (4P)
- net Out_P2_B8: now also J?.16 (4K)
- net Out_P2_Down: now also J?.2 (Down)
- net Out_P2_Left: now also J?.4 (Left)
- net Out_P2_Right: now also J?.3 (Right)
- net Out_P2_Start: now also J?.7 (Start/Opt)
- net Out_P2_Up: now also J?.1 (Up)
Other:
- note added: "Note:\nSW_Bypass_Auto is a hardware switch\nto disable all 'advanced' input processing\n(autofire, macros, etc.). It still allows\nremapping to be used.\nThis is a convenience feature to quickly\nenable/disable the aspects of the device\nthat might be considered 'unfair', sort of\nlike a 'tournament mode' toggle."
