File: kicad/ESP-In-De_JAMMA_THT/ESP-In-De_JAMMA_THT.kicad_sch (KiCad schematic)
At the start: 50 parts

Commit message: added Coin remapping
Connections:
- net DIP1: now also RN?.8 (R7), U?.5 (D6); no longer RN?.7 (R6), U?.4 (D5)
- net DIP2: now also RN?.9 (R8), U?.6 (D7); no longer RN?.8 (R7), U?.5 (D6)
- net DIP3: now also RN?.8 (R7), U?.5 (D6); no longer RN?.9 (R8), U?.6 (D7)
- net DIP4: now also RN?.9 (R8), U?.6 (D7); no longer RN?.7 (R6), U?.4 (D5)
- net DIP5: no longer RN?.8 (R7), U?.5 (D6)
- net DIP6: no longer RN?.9 (R8), U?.6 (D7)
- net GND: no longer U?.5 (3A), U?.9 (4A)
- net O_P2_B1: now also U?.4 (~{2Y}); no longer U?.2 (~{1Y})
- net O_P2_B2: now also U?.6 (~{3Y}); no longer U?.4 (~{2Y})
- net O_P2_B3: now also U?.8 (~{4Y}); no longer U?.6 (~{3Y})
- net O_P2_B4: now also U?.10 (~{5Y}); no longer U?.8 (~{4Y})
- net O_P2_B5: now also U?.12 (~{6Y}); no longer U?.10 (~{5Y})
- net O_P2_B6: now also U?.2 (~{1Y}); no longer U?.12 (~{6Y})
- net O_P2_B7: now also U?.4 (~{2Y}); no longer U?.2 (~{1Y})
- net O_P2_B8: now also U?.6 (~{3Y}); no longer U?.4 (~{2Y})
- net O_P2_Down: now also U?.8 (~{4Y}); no longer U?.6 (~{3Y})
- net O_P2_Left: now also U?.10 (~{5Y}); no longer U?.8 (~{4Y})
- net O_P2_Right: now also U?.12 (~{6Y}); no longer U?.10 (~{5Y})
- net O_P2_Start: now also U?.2 (~{1Y}); no longer U?.12 (~{6Y})
- net O_P2_Up: now also U?.6 (~{3Y}); no longer U?.4 (~{2Y})
- net at U?.5 (QF): now also U?.3 (2A)
- net at U?.1 (QB): now also U?.9 (4A); no longer U?.5 (3A)
- net at U?.15 (QA): now also U?.5 (3A); no longer U?.3 (2A)
- net at U?.2 (QC): now also U?.11 (5A); no longer U?.9 (4A)
- net at U?.3 (QD): now also U?.13 (6A); no longer U?.11 (5A)
- net at U?.4 (QE): now also U?.1 (1A); no longer U?.13 (6A)
- net at U?.5 (QF): now also U?.3 (2A); no longer U?.1 (1A)
- net at U?.6 (QG): now also U?.5 (3A); no longer U?.3 (2A)
- net at U?.7 (QH): now also U?.9 (4A); no longer U?.5 (3A)
- net at U?.1 (QB): now also U?.13 (6A); no longer U?.11 (5A)
- net at U?.15 (QA): now also U?.11 (5A); no longer U?.9 (4A)
- net at U?.2 (QC): now also U?.1 (1A); no longer U?.13 (6A)
- net at U?.3 (QD): now also U?.3 (2A); no longer U?.1 (1A)
- net at U?.4 (QE): now also U?.5 (3A); no longer U?.3 (2A)
- net at U?.5 (QF): now also U?.9 (4A)
- net O_P2_Coin: now reaches U?.8 (~{4Y})
- net O_P2_Coin: now also J?.T (Coin_2)
- net Coin1 renamed I_P1_Coin
- net I_P1_Coin: now also RN?.7 (R6), U?.4 (D5); no longer J?.16 (Coin_1)
- net Coin2 renamed I_P2_Coin
- net I_P2_Coin: now also RN?.7 (R6), U?.4 (D5); no longer J?.T (Coin_2)
- new net O_P1_Coin: J?.16 (Coin_1), U?.4 (~{2Y})
- no-connect marks 25 -> 22
