File: kicad/ESP-In-De_JAMMA_THT/ESP-In-De_JAMMA_THT.kicad_sch (KiCad schematic)
At the start: 50 parts

Commit message: Add kick connections, update encoder pullups
Parts:
- removed R? (x3): 10k, symbol Device:R_Small
- removed SW?: SW_DIP_x06, symbol Switch:SW_DIP_x06
- added J?: Game Board Kick Header, symbol Connector_Generic:Conn_01x08
- added SW? (x2): B5_Enable, symbol Switch:SW_DPDT_x2
- added SW?: SW_DIP_x04, symbol Switch:SW_DIP_x04
Connections:
- net DIP1: now also SW?.8
- net DIP2: now also SW?.7
- net DIP3: now also SW?.6
- net DIP4: now also SW?.5
- net GND: now also J?.8 (Pin_8), SW?.1, SW?.2, SW?.3, SW?.4
- net O_P1_B5: now also SW?.1 (A)
- net O_P1_B6: no longer U?.10 (~{5Y})
- net O_P1_B7: no longer U?.12 (~{6Y})
- net O_P1_B8: no longer U?.2 (~{1Y})
- net O_P2_B5: now also SW?.4 (A)
- net O_P2_B6: no longer U?.2 (~{1Y})
- net O_P2_B7: no longer U?.4 (~{2Y})
- net O_P2_B8: no longer U?.6 (~{3Y})
- net O_JAMMA_25: now reaches J?.26 (OPT_P1_Button_5)
- net O_JAMMA_25: now also SW?.2 (B)
- net O_JAMMA_d: now reaches J?.d (OPT_P2_Button_5)
- net O_JAMMA_d: now also SW?.5 (B)
- new net O_P1_K1: J?.1 (Pin_1), U?.10 (~{5Y})
- new net O_P1_K2: J?.2 (Pin_2), U?.12 (~{6Y})
- new net O_P1_K3: J?.3 (Pin_3), U?.2 (~{1Y})
- new net O_P2_K1: J?.4 (Pin_4), U?.2 (~{1Y})
- new net O_P2_K2: J?.5 (Pin_5), U?.4 (~{2Y})
- new net O_P2_K3: J?.6 (Pin_6), U?.6 (~{3Y})
- no-connect marks 22 -> 23
Other:
- note added: "DPDT switch to select N/C or Button 5 on JAMMA edge"
- note added: "Game Board Connections"
- note added: "SW1 | Bypass Auto SW2 | SW3 | SW4 |"
- note added: "Uses internal GPIO pullups"
- note removed: "SW1 | Bypass Auto SW2 | SW3 | SW4 | SW5 | SW6 |"

Commit message: Minor tweak to sch
Parts:
- added J?: Sync In, symbol Connector:Conn_Coaxial
- added J?: Sync Out, symbol Connector:Conn_Coaxial
- added R?: 75, symbol Device:R_Small
- added SW?: SW_SPDT, symbol Switch:SW_SPDT
Connections:
- net GND: now also J?.2 (Ext), J?.2 (Ext), R?.2
- new net: R?.1, SW?.3 (C)
- new net External_Sync: J?.1 (In), J?.1 (In), SW?.2 (B)
- no-connect marks 23 -> 24
Other:
- note added: "BNC external sync input and loop. Termination switch. Adapted from https://community.lzxindustries.net/t/ best-way-to-do-rca-sync-thru/2287/2"
